File: 6-axis pcb/6-axis pcb.kicad_pcb (KiCad board)
At the start: 2 copper layers, 80 x 140 mm, 28 parts, among them J1 Conn_01x04_Pin, J2 Conn_01x04_Pin, J3 Conn_01x04_Pin, J4 Conn_01x04_Pin, J5 Conn_01x04_Pin, J6 Conn_01x04_Pin, U1 ESP32-C6-DEVKITC-1-N8

Commit message: Move to PC
Parts:
- moved A6 23.5 mm to (68.3, 91.8), turned to 90 degrees
- moved U2 11.9 mm to (61.5, 76.1), turned to 180 degrees
- moved ENCODER4I2C1 4.51 mm to (59.8, 36.8), turned to 180 degrees
Routing:
- net +12V: track 0.00 -> 123.3 mm
- net +5V: track 0.00 -> 92.8 mm
- net /SC1: track 0.00 -> 27.9 mm
- net Net-(A2-1B): track 0.00 -> 22.5 mm
- net Net-(A2-2A): track 0.00 -> 22.2 mm
- net Net-(A6-1B): track 0.00 -> 21.9 mm
- net Net-(A4-1B): track 0.00 -> 21.9 mm
- net Net-(A3-1A): track 0.00 -> 21.9 mm
- net Net-(A4-2A): track 0.00 -> 21.8 mm
- net Net-(A3-1B): track 0.00 -> 21.6 mm
- net Net-(A5-1B): track 0.00 -> 21.3 mm
- net Net-(A1-2B): track 0.00 -> 19.9 mm
- net Net-(A2-1A): track 0.00 -> 18.3 mm
- net Net-(A6-1A): track 0.00 -> 17.7 mm
- net Net-(A4-1A): track 0.00 -> 17.7 mm
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
Commit message: Move to Laptop
Parts:
- added C2: EEUFK1V102S, 5x12 electrolytic capacitor:CAPPRD750W80D1600H1500, F.Cu at (66.8, 109.0)
- added C3: EEUFK1V102S, 5x12 electrolytic capacitor:CAPPRD750W80D1600H1500, F.Cu at (61.5, 126.0)
- added C4: EEUFK1V102S, 5x12 electrolytic capacitor:CAPPRD750W80D1600H1500, F.Cu at (68.5, 143.0)
- added C5: EEUFK1V102S, 5x12 electrolytic capacitor:CAPPRD750W80D1600H1500, F.Cu at (69.0, 161.5)
- added C6: EEUFK1V102S, 5x12 electrolytic capacitor:CAPPRD750W80D1600H1500, F.Cu at (74.5, 66.5)
- added C7: EEUFK1V102S, 5x12 electrolytic capacitor:CAPPRD750W80D1600H1500, F.Cu at (46.2, 100.5)
- moved ArmDifferential1 76.0 mm to (68.4, 90.2)
- moved Zwrist1 75.9 mm to (79.1, 166.8)
- moved J6 75.7 mm to (102.0, 163.5)
- moved J5 74.5 mm to (92.0, 88.5)
- moved ENCODER2I2C1 48.4 mm to (55.0, 37.0), turned to 0 degrees
- moved ENCODER4I2C1 47.0 mm to (32.0, 74.8), turned to -90 degrees
- moved J7 28.5 mm to (84.0, 55.6), turned to 180 degrees
- moved U2 2.00 mm to (61.2, 74.2)
- moved J1 1.80 mm to (41.5, 83.5)
- moved Basestepper1 1.50 mm to (45.6, 90.3)
- moved ENCODER5I2C1 0.25 mm to (79.2, 37.0)
- renumbered A3 to ARM1, A5 to ArmDifferential1, A1 to Basestepper1, A2 to Shoulder1, A4 to Wrist1, A6 to Zwrist1
Connections:
- ARM1 pad 13: unconnected-(A3-~{RESET}-Pad13) -> Net-(ARM1-~{RESET})
- ARM1 pad 14: Net-(A3-~{ENABLE}) -> Net-(ARM1-~{RESET})
- ARM1 pad 9: Net-(A3-~{ENABLE}) -> unconnected-(ARM1-~{ENABLE}-Pad9)
- ArmDifferential1 pad 13: unconnected-(A5-~{RESET}-Pad13) -> Net-(ArmDifferential1-~{RESET})
- ArmDifferential1 pad 14: Net-(A5-~{ENABLE}) -> Net-(ArmDifferential1-~{RESET})
- ArmDifferential1 pad 9: Net-(A5-~{ENABLE}) -> unconnected-(ArmDifferential1-~{ENABLE}-Pad9)
- Basestepper1 pad 13: unconnected-(A1-~{RESET}-Pad13) -> Net-(Basestepper1-~{RESET})
- Basestepper1 pad 14: Net-(A1-~{ENABLE}) -> Net-(Basestepper1-~{RESET})
- Basestepper1 pad 9: Net-(A1-~{ENABLE}) -> unconnected-(Basestepper1-~{ENABLE}-Pad9)
- J7 pad 1: +12V -> +5V
- J7 pad 4: +5V -> +12V
- Shoulder1 pad 13: unconnected-(A2-~{RESET}-Pad13) -> Net-(Shoulder1-~{RESET})
- Shoulder1 pad 14: Net-(A2-~{ENABLE}) -> Net-(Shoulder1-~{RESET})
- Shoulder1 pad 9: Net-(A2-~{ENABLE}) -> unconnected-(Shoulder1-~{ENABLE}-Pad9)
- Wrist1 pad 13: unconnected-(A4-~{RESET}-Pad13) -> Net-(Wrist1-~{RESET})
- Wrist1 pad 14: Net-(A4-~{ENABLE}) -> Net-(Wrist1-~{RESET})
- Wrist1 pad 9: Net-(A4-~{ENABLE}) -> unconnected-(Wrist1-~{ENABLE}-Pad9)
- Zwrist1 pad 13: unconnected-(A6-~{RESET}-Pad13) -> Net-(Zwrist1-~{RESET})
- Zwrist1 pad 14: Net-(A6-~{ENABLE}) -> Net-(Zwrist1-~{RESET})
- Zwrist1 pad 9: Net-(A6-~{ENABLE}) -> unconnected-(Zwrist1-~{ENABLE}-Pad9)
Routing:
- net GND: track 0.00 -> 636.1 mm, vias 0 -> 5
- net +12V: track 123.3 -> 350.6 mm, vias 0 -> 1
- net +5V: track 92.8 -> 215.8 mm, vias 0 -> 1
- net /SD0: track 0.00 -> 108.5 mm
- net /SCL: track 0.00 -> 80.3 mm
- net /SDA: track 0.00 -> 73.7 mm
- net /SC5: track 0.00 -> 69.2 mm, vias 0 -> 1
- net /GPIO11: track 0.00 -> 68.7 mm
- net /SD5: track 0.00 -> 67.9 mm, vias 0 -> 1
- net /GPIO1: track 0.00 -> 66.4 mm
- net /GPIO0: track 0.00 -> 62.8 mm
- net /<NO NET>: track 3.32 -> 66.1 mm, vias 0 -> 1
- net /SC0: track 0.00 -> 61.6 mm
- net /GPIO10: track 0.00 -> 59.0 mm
- net /GPIO23: track 0.00 -> 58.4 mm, vias 0 -> 1
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Other:
- board text added: "12V"
- board text added: "3.3 V"
- board text added: "3.3v"
- board text added: "5V"
- board text added: "5v Buck"
- board text added: "EN"
- board text added: "ESP32 C6"
- board text added: "GND"
- board text added: "SC0"
- board text added: "SC1"
- board text added: "SC2"
- board text added: "SC3"
- board text added: "SC4"
- board text added: "SC5"
- board text added: "SD0"
- board text added: "SD1"
- board text added: "SD2"
- board text added: "SD3"
- board text added: "SD4"
- board text added: "SD5"

Commit message: Move to pc
Routing:
- net GND: track 636.1 -> 569.7 mm
- net +3.3V: track 255.8 -> 221.4 mm
- net /SC5: track 69.2 -> 45.8 mm
- net /SD5: track 67.9 -> 55.9 mm

Commit message: Final Commit
Ready for manufacturing
Parts:
- removed C6: EEUFK1V102S, 5x12 electrolytic capacitor:CAPPRD750W80D1600H1500
- removed MainPoweRails1: Screw_Terminal_01x02, TerminalBlock:TerminalBlock_MaiXu_MX126-5.0-02P_1x02_P5.00mm
- removed U2: ~, I2C Breakout:Untitled
- added Battery1: Screw_Terminal_01x02, TerminalBlock:TerminalBlock_MaiXu_MX126-5.0-02P_1x02_P5.00mm, F.Cu at (30.8, 128.6)
- added Ce1: EEUFK1V102S, Capacitor_THT:CP_Radial_Tantal_D6.0mm_P2.50mm, F.Cu at (70.4, 106.3)
- added D1: D, Diode_THT:D_5KPW_P12.70mm_Horizontal, F.Cu at (58.4, 73.0)
- added Switch1: Screw_Terminal_01x02, TerminalBlock:TerminalBlock_MaiXu_MX126-5.0-02P_1x02_P5.00mm, F.Cu at (30.7, 140.6)
- added TCA 9548: ~, I2C Breakout:Untitled, F.Cu at (80.7, 111.4)
- C2, C3, C4, C5, C7: footprint 5x12 electrolytic capacitor:CAPPRD750W80D1600H1500 -> Capacitor_THT:CP_Radial_Tantal_D6.0mm_P2.50mm
- moved J6 129.2 mm to (57.9, 42.0), turned to 90 degrees
- moved Encoder3PWR1 123.4 mm to (90.0, 151.1)
- moved Zwrist1 122.1 mm to (70.5, 45.1), turned to -90 degrees
- moved ENCODER2I2C1 114.0 mm to (53.9, 151.0)
- moved ENCODER3I2C1 106.9 mm to (78.0, 151.0), turned to 0 degrees
- moved J4 105.8 mm to (81.0, 42.0), turned to 90 degrees
- moved Wrist1 104.9 mm to (93.2, 45.1), turned to -90 degrees
- moved C4 103.4 mm to (73.0, 39.7), turned to 0 degrees
- moved Encoder4PWR1 97.8 mm to (100.1, 129.2), turned to 90 degrees
- moved ENCODER4I2C1 95.0 mm to (100.2, 141.0), turned to 90 degrees
- moved Encoder2PWR1 90.7 mm to (66.1, 151.0), turned to 0 degrees
- moved C3 87.0 mm to (50.4, 39.7), turned to 0 degrees
- moved C2 84.5 mm to (27.3, 34.2), turned to 0 degrees
- moved ENCODER5I2C1 82.6 mm to (100.1, 116.9), turned to 90 degrees
- moved J7 76.7 mm to (28.1, 108.2), turned to 0 degrees
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Connections:
- ARM1 pad 2: +5V -> +3.3V
- ArmDifferential1 pad 15: /GPIO23 -> /GPIO15
- ArmDifferential1 pad 16: /GPIO15 -> /GPIO23
- ArmDifferential1 pad 2: +5V -> +3.3V
- Basestepper1 pad 2: +5V -> +3.3V
- ENCODER3I2C1 pad 1: /SC2 -> /SD2
- ENCODER3I2C1 pad 2: /SD2 -> /SC2
- ENCODER4I2C1 pad 1: /SC3 -> /SD3
- ENCODER4I2C1 pad 2: /SD3 -> /SC3
- ENCODER5I2C1 pad 1: /SC4 -> /SD4
- ENCODER5I2C1 pad 2: /<NO NET> -> /SC4
- ENCODER6I2C1 pad 1: /SC5 -> /SD5
- ENCODER6I2C1 pad 2: /SD5 -> /SC5
- Shoulder1 pad 2: +5V -> +3.3V
- U1 pad J1_14: +5V -> Net-(D1-K)
- Wrist1 pad 2: +5V -> +3.3V
- Zwrist1 pad 15: /GPIO21 -> /GPIO22
- Zwrist1 pad 16: /GPIO22 -> /GPIO21
- Zwrist1 pad 2: +5V -> +3.3V
Routing:
- net +3.3V: track 221.4 -> 444.8 mm, vias 0 -> 2
- net +5V: track 215.8 -> 46.2 mm, vias 1 -> 0
- net +12V: track 350.6 -> 264.1 mm, vias 1 -> 0
- net /<NO NET>: track 66.1 -> 0.00 mm, vias 1 -> 0
- net /GPIO1: track 66.4 -> 4.66 mm
- net /GPIO0: track 62.8 -> 4.66 mm
- net /GPIO23: track 58.4 -> 5.04 mm, vias 1 -> 0
- net /SD0: track 108.5 -> 56.0 mm
- net /GPIO11: track 68.7 -> 18.5 mm
- net /GPIO15: track 54.8 -> 5.04 mm, vias 1 -> 0
- net /GPIO5: track 62.4 -> 12.9 mm
- net /SD4: track 0.00 -> 45.5 mm
- net /GPIO4: track 54.5 -> 12.9 mm
- net /GPIO10: track 59.0 -> 18.5 mm
- net /SC1: track 8.37 -> 41.4 mm
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- added copper zone on F.Cu, net +12V
- added copper zone on B.Cu, net GND
Other:
- outline, holes or cut-outs redrawn
- board text added: "3.3V"
- board text added: "Common"
- board text added: "NO"
- board text added: "VBat"
- board text removed: "3.3 V"
- board text removed: "5V"
- board text removed: "5v Buck"
- board text removed: "EN"
- board text removed: "ESP32 C6"
