File: 6-axis pcb/6-axis pcb.kicad_sch (KiCad schematic)
At the start: 28 parts, among them J1 Conn_01x04_Pin, J2 Conn_01x04_Pin, J3 Conn_01x04_Pin, J4 Conn_01x04_Pin, J5 Conn_01x04_Pin, J6 Conn_01x04_Pin, U1 ESP32-C6-DEVKITC-1-N8

Commit message: Move to PC
Other:
- moved on the sheet: ENCODER5I2C1
Changed lines of the file:
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@@
 	(wire
 		(pts
-			(xy 71.12 251.46) (xy 85.09 251.46)
+			(xy 71.12 251.46) (xy 87.63 251.46)
 		)
 		(stroke
@@
 	(wire
 		(pts
-			(xy 71.12 248.92) (xy 85.09 248.92)
+			(xy 71.12 248.92) (xy 87.63 248.92)
 		)
 		(stroke
@@
 	(symbol
 		(lib_id "Connector:Screw_Terminal_01x02")
-		(at 90.17 248.92 0)
+		(at 92.71 248.92 0)
 		(unit 1)
 		(body_style 1)
@@
 		(dnp no)
 		(property "Reference" "ENCODER5I2C1"
-			(at 92.71 248.9199 0)
+			(at 95.25 248.9199 0)
 			(show_name no)
 			(do_not_autoplace no)
@@
 		)
 		(property "Value" "Screw_Terminal_01x02"
-			(at 92.71 251.4599 90)
+			(at 95.25 251.4599 0)
 			(show_name no)
 			(do_not_autoplace no)
@@
 		)
 		(property "Footprint" "TerminalBlock:TerminalBlock_MaiXu_MX126-5.0-02P_1x02_P5.00mm"
-			(at 90.17 248.92 0)
+			(at 92.71 248.92 0)
 			(hide yes)
 			(show_name no)
@@
 		)
 		(property "Datasheet" ""
-			(at 90.17 248.92 0)
+			(at 92.71 248.92 0)
 			(hide yes)
 			(show_name no)
@@
 		)
 		(property "Description" "Generic screw terminal, single row, 01x02, script generated (kicad-library-utils/schlib/autogen/connector/)"
-			(at 90.17 248.92 0)
-			(hide yes)
-			(show_name no)
+			(at 92.71 248.92 0)
+			(hide yes)
+			(show_name no)

Commit message: Move to Laptop
Parts:
- removed A3: Pololu_Breakout_A4988, Module:Pololu_Breakout-16_15.2x20.3mm, symbol Driver_Motor:Pololu_Breakout_A4988
- added ARM1: Pololu_Breakout_A4988, Module:Pololu_Breakout-16_15.2x20.3mm, symbol Driver_Motor:Pololu_Breakout_A4988
- added C2, C3, C4, C5, C6, C7: EEUFK1V102S, 5x12 electrolytic capacitor:CAPPRD750W80D1600H1500, symbol 6x12 electrolytic capacitor:EEUFK1V102S
- added MainPoweRails2: Screw_Terminal_01x02, TerminalBlock:TerminalBlock_MaiXu_MX126-5.0-02P_1x02_P5.00mm, symbol Connector:Screw_Terminal_01x02
- renumbered A5 to ArmDifferential1, A1 to Basestepper1, A2 to Shoulder1, A4 to Wrist1, A6 to Zwrist1
Connections:
- net +12V: now also J7.4 (IN+), ARM1.8 (VMOT), C2.P, C3.P, C4.P, C5.P, C6.P, C7.P; no longer J7.1 (OUT+)
- net +5V: now also J7.1 (OUT+), ARM1.2 (VDD); no longer J7.4 (IN+)
- net GND: now also ARM1.1 (GND), ARM1.7 (GND), C2.N, C3.N, C4.N, C5.N, C6.N, C7.N, MainPoweRails2.2 (Pin_2)
- net GPIO10: now also ARM1.16 (DIR)
- net GPIO11: now also ARM1.15 (STEP)
- net SD4: now reaches ENCODER5I2C1.2 (Pin_2), U2.17 (SD4)
- net at J3.1 (Pin_1): now also ARM1.6 (2B)
- net at J3.2 (Pin_2): now also ARM1.4 (1A)
- net at J3.3 (Pin_3): now also ARM1.5 (2A)
- net at J3.4 (Pin_4): now also ARM1.3 (1B)
- new net: ARM1.13 (~{RESET}), ARM1.14 (~{SLEEP})
- no-connect marks 0 -> 42
Other:
- moved on the sheet: J3

Commit message: Move to pc
Parts:
- removed MainPoweRails2: Screw_Terminal_01x02, TerminalBlock:TerminalBlock_MaiXu_MX126-5.0-02P_1x02_P5.00mm, symbol Connector:Screw_Terminal_01x02
- added J10, J9: Screw_Terminal_01x02, TerminalBlock:TerminalBlock_MaiXu_MX126-5.0-02P_1x02_P5.00mm, symbol Connector:Screw_Terminal_01x02
Connections:
- net +12V: now also J9.2 (Pin_2); no longer MainPoweRails1.1 (Pin_1)
- new net LED+: J10.1 (Pin_1)
- new net LED-: J10.2 (Pin_2)
- new net VBattery: J9.1 (Pin_1), MainPoweRails1.1 (Pin_1)
Other:
- note added: "NO"

Commit message: Final Commit
Ready for manufacturing
Parts:
- removed J10, J9: Screw_Terminal_01x02, TerminalBlock:TerminalBlock_MaiXu_MX126-5.0-02P_1x02_P5.00mm, symbol Connector:Screw_Terminal_01x02
- added D1: D, Diode_THT:D_5KPW_P12.70mm_Horizontal, symbol Device:D
- added Switch1: Screw_Terminal_01x02, TerminalBlock:TerminalBlock_MaiXu_MX126-5.0-02P_1x02_P5.00mm, symbol Connector:Screw_Terminal_01x02
- C2, C3, C4, C5, C7: footprint 5x12 electrolytic capacitor:CAPPRD750W80D1600H1500 -> Capacitor_THT:CP_Radial_Tantal_D6.0mm_P2.50mm
- Ce1: renamed from C6; footprint 5x12 electrolytic capacitor:CAPPRD750W80D1600H1500 -> Capacitor_THT:CP_Radial_Tantal_D6.0mm_P2.50mm
- renumbered MainPoweRails1 to Battery1
Connections:
- net +12V: now also C2.1, C3.1, C4.1, C5.1, C7.1, Ce1.1, Switch1.1 (Pin_1); no longer C2.P, C3.P, C4.P, C5.P, C7.P, Ce1.P
- net +3.3V: now also ARM1.2 (VDD), ArmDifferential1.2 (VDD), Basestepper1.2 (VDD), Shoulder1.2 (VDD), Wrist1.2 (VDD), Zwrist1.2 (VDD)
- net +5V: now also D1.2 (A); no longer ARM1.2 (VDD), ArmDifferential1.2 (VDD), Basestepper1.2 (VDD), Shoulder1.2 (VDD), U1.J1_14 (VCC_5V), Wrist1.2 (VDD), Zwrist1.2 (VDD)
- net GND: now also C2.2, C3.2, C4.2, C5.2, C7.2, Ce1.2; no longer C2.N, C3.N, C4.N, C5.N, C7.N, Ce1.N
- net GPIO15: now also ArmDifferential1.15 (STEP); no longer ArmDifferential1.16 (DIR)
- net GPIO21: now also Zwrist1.16 (DIR); no longer Zwrist1.15 (STEP)
- net GPIO22: now also Zwrist1.15 (STEP); no longer Zwrist1.16 (DIR)
- net GPIO23: now also ArmDifferential1.16 (DIR); no longer ArmDifferential1.15 (STEP)
- net SC2: now also ENCODER3I2C1.2 (Pin_2); no longer ENCODER3I2C1.1 (Pin_1)
- net SC3: now also ENCODER4I2C1.2 (Pin_2); no longer ENCODER4I2C1.1 (Pin_1)
- net SC4: now also ENCODER5I2C1.2 (Pin_2); no longer ENCODER5I2C1.1 (Pin_1)
- net SC5: now also ENCODER6I2C1.2 (Pin_2); no longer ENCODER6I2C1.1 (Pin_1)
- net SD2: now also ENCODER3I2C1.1 (Pin_1); no longer ENCODER3I2C1.2 (Pin_2)
- net SD3: now also ENCODER4I2C1.1 (Pin_1); no longer ENCODER4I2C1.2 (Pin_2)
- net SD4: now also ENCODER5I2C1.1 (Pin_1); no longer ENCODER5I2C1.2 (Pin_2)
- net SD5: now also ENCODER6I2C1.1 (Pin_1); no longer ENCODER6I2C1.2 (Pin_2)
- net VBattery: now also Switch1.2 (Pin_2)
- new net: D1.1 (K), U1.J1_14 (VCC_5V)
- no-connect marks 42 -> 43
Other:
- note removed: "NO"
